Commit message: remove directory

File: src/UR3e_RG2_ER5/UR3e_RG2_ER5_vision/box.urdf (robot description, URDF)
Before this commit: robot simple_box, 1 links, 0 joints
Links:
- link my_box: geometry collision box size=0.05 0.05 0.05; visual box size=0.05 0.05 0.05

File: src/UR3e_RG2_ER5/UR3e_RG2_ER5_vision/cylinder.urdf (robot description, URDF)
Before this commit: robot simple_cylinder, 1 links, 0 joints
Links:
- link cylinder: geometry collision cylinder length=0.05 radius=0.05; visual cylinder length=0.05 radius=0.05
